Commit message: Resolved errors with controlling robot, pid needs to be tuned

File: delta_robot_support/urdf/delta_robot.urdf.xacro (robot description, xacro)
@@ -17,5 +17,5 @@
   <xacro:property name="width_lleg" value="0.002" /> <!-- low leg width -->
   <xacro:property name="mass_con" value="0.0173" /> <!-- connector mass-->
-  <xacro:property name="namespace" value="delta" />
+  <xacro:property name="namespace" value="delta_robot" />
   <xacro:macro name="default_inertial2" params="mass length width">
 	 <inertia ixx="${1/12*mass*(width*width+length*length)}" ixy="0.0" ixz="0.0"
@@ -131,5 +131,5 @@
     	<parent link="link_0"/>
     	<child link="uleg_1"/>
-      <limit effort="20" velocity="1.0" lower="-1.1" upper="1.1" />
+      <limit effort="20" velocity="1.0" lower="-2.1" upper="2.1" />
       <axis xyz="1 0 0"/>
     </joint>
@@ -138,5 +138,5 @@
     	<parent link="link_0"/>
     	<child link="uleg_2"/>
-      <limit effort="20" velocity="1.0" lower="-1.1" upper="1.1" />
+      <limit effort="20" velocity="1.0" lower="-2.1" upper="2.1" />
       <axis xyz="1 0 0"/>
     </joint>
@@ -145,5 +145,5 @@
     	<parent link="link_0"/>
     	<child link="uleg_3"/>
-      <limit effort="20" velocity="1.0" lower="-1.1" upper="1.1" />
+      <limit effort="20" velocity="1.0" lower="-2.1" upper="2.1" />
       <axis xyz="1 0 0"/>
     </joint>
@@ -661,5 +661,5 @@
 <!-- Joins trabsmisions motors for gazebo  -->
 <!-- ****************************************************************** -->
-       <transmission name="motor1_trans">
+       <!-- <transmission name="motor1_trans">
          <type>transmission_interface/SimpleTransmission</type>
          <joint name="link_0_JOINT_1">
@@ -711,6 +711,6 @@
           <stopKp value="100000000.0" />
           <fudgeFactor value="0.5" />
-       </gazebo>
-       <gazebo>
+       </gazebo> -->
+       <!-- <gazebo>
            <gazebo_ros_controller_manager name="gazebo_ros_controller_manager" plugin="libgazebo_ros_controller_manager.so">
                 <alwaysOn>true</alwaysOn>
@@ -720,5 +720,5 @@
                 <audio name="gazebo_ros_controller_manager_dummy_iface" />
            </gazebo_ros_controller_manager>
-      </gazebo>
+      </gazebo> -->
 <!--
       <plugin name="copter_arm_sim_plugin" filename="libgazebo_ros_control.so">
@@ -726,5 +726,5 @@
       </plugin>
 -->
-        <gazebo>
+        <!-- <gazebo>
             <plugin name="gazebo_ros_f3d" filename="libgazebo_ros_f3d.so">
                 <alwaysOn>true</alwaysOn>
@@ -734,4 +734,36 @@
                 <frameName>${namespace}/low_base</frameName>
             </plugin>
-        </gazebo>
+        </gazebo> -->
+    <transmission name="motor1_trans">
+      <type>transmission_interface/SimpleTransmission</type>
+      <actuator name="motor1">
+        <mechanicalReduction>1</mechanicalReduction>
+      </actuator>
+      <joint name="link_0_JOINT_1">
+        <hardwareInterface>hardware_interface/PositionJointInterface</hardwareInterface>
+      </joint>
+    </transmission>
+    <transmission name="motor2_trans">
+      <type>transmission_interface/SimpleTransmission</type>
+      <actuator name="motor2">
+        <mechanicalReduction>1</mechanicalReduction>
+      </actuator>
+      <joint name="link_0_JOINT_2">
+        <hardwareInterface>hardware_interface/PositionJointInterface</hardwareInterface>
+      </joint>
+    </transmission>
+    <transmission name="motor3_trans">
+      <type>transmission_interface/SimpleTransmission</type>
+      <actuator name="motor3">
+        <mechanicalReduction>1</mechanicalReduction>
+      </actuator>
+      <joint name="link_0_JOINT_3">
+        <hardwareInterface>hardware_interface/PositionJointInterface</hardwareInterface>
+      </joint>
+    </transmission>
+    <gazebo>
+      <plugin name="gazebo_ros_control" filename="libgazebo_ros_control.so">
+         <robotNamespace>/</robotNamespace>
+       </plugin>
+    </gazebo>
 </robot>

Commit message: Add files via upload

File: delta_robot_support/urdf/delta_robot.urdf.xacro (robot description, xacro)
@@ -1,6 +1,9 @@
 <?xml version="1.0"?>
 <robot name="delta_robot" xmlns:xacro="http://www.ros.org/wiki/xacro">
-  <xacro:property name="PI" value="3.1415926535897931"/>
-  <xacro:property name="width" value="0.01" /> <!-- all links -->
+  	<xacro:property name="PI" value="3.1415926535897931"/>
+  	<xacro:property name="width" value="0.01" /> <!-- all links -->
+  	<xacro:property name="u" value="0.075" /> <!-- Radius of Base -->
+	<xacro:property name="ul" value="0.1" /> <!-- Length of Upper Leg -->
+	<xacro:property name="ll" value="0.15" /> <!-- Length of Lower Leg -->
   <xacro:property name="width_m" value="0.01" /> <!-- all links -->
   <xacro:property name="length_m" value="0.03" /> <!-- all links -->
@@ -14,199 +17,172 @@
   <xacro:property name="width_uleg" value="0.05" /> <!-- upper leg width -->
   <xacro:property name="mass_lleg" value="0.04" /> <!-- low leg mass-->
-  <xacro:property name="length_lleg" value="0.51" /> <!-- low leg length-->
+  <xacro:property name="length_lleg" value="0.2" /> <!-- low leg length-->
   <xacro:property name="width_lleg" value="0.002" /> <!-- low leg width -->
   <xacro:property name="mass_con" value="0.0173" /> <!-- connector mass-->
   <xacro:property name="namespace" value="delta_robot" />
-  <xacro:macro name="default_inertial2" params="mass length width">
-	 <inertia ixx="${1/12*mass*(width*width+length*length)}" ixy="0.0" ixz="0.0"
-	  	  iyy="${1/12*mass*(width*width+length*length)}" iyz="0.0"
-	 	  izz="${1/12*mass*(width*width+width*width)}"/>
-  </xacro:macro>
-  <xacro:macro name="default_inertial3" params="mass length width">
-	 <inertia ixx="${1/12*mass*(width*width+length*length)}" ixy="0.0" ixz="0.0"
-	  	  iyy="${1/12*mass*(width*width+length*length)}" iyz="0.0"
-	 	  izz="${1/12*mass*(length*length+length*length)}"/>
-  </xacro:macro>
-  <gazebo>
-     <plugin name="my_plugin" filename="libcontact.so"/>
-     <plugin filename="libgazebo_ros_control.so" name="gazebo_ros_control">
-       <robotNamespace>/${namespace}</robotNamespace>
-     </plugin>
- 	   <self_collide>true</self_collide>
-     <enable_wind>false</enable_wind>
-   </gazebo>
-   <link name="world"/>
-<!-- Base superior -->
-   <joint name="base" type="fixed">
- 	     <parent link="world"/>
- 	     <child link="link_0"/>
-       <axis xyz="0 0 0"/>
-       <origin xyz="0 0 ${-distance_arm_uav+distance_ground}" rpy="0 0 1.57"/>
-   </joint>
-   <gazebo reference="link_w_JOINT_w2">
- 	    <physics>
-   		 <ode>
-   	    <provide_feedback>true</provide_feedback>
-   		 </ode>
- 	    </physics>
- 	 </gazebo>
-   <link name="link_0">
-      <inertial>
-        <origin xyz="-0.0 -0.0 -0.0" rpy="0 0 0"/>
-        <mass value="${mass_base}"/>
-        <xacro:default_inertial3 mass="${mass_base}" length="${length_base}" width="${width_m}" />
-      </inertial>
-      <visual>
-        <origin xyz="-0.147 -0.085 -0.01" rpy="0 0 0"/>
-   	    <geometry>
-          <mesh filename="package://delta_robot_support/urdf/meshes/fixed_base2.dae" scale="0.001 0.001 0.001" />
-        </geometry>
-      </visual>
-      <visual>
-        <origin xyz="-0.0 0 ${distance_arm_uav/2}" rpy="0 0 0"/>
-        <geometry>
-   	      <box size="0.05 0.05 ${distance_arm_uav}  "/>
-        </geometry>
-      </visual>
-      <collision>
-        <origin xyz="-0.147 -0.085 -0.01" rpy="0 0 0"/>
-        <geometry>
-            <mesh filename="package://delta_robot_support/urdf/meshes/fixed_base2.dae" scale="0.001 0.001 0.001" />
-        </geometry>
-      </collision>
-    </link>
-    <gazebo reference="link_0">
-      <visual>
-        <material>
-          <script>
-            <uri>file://media/materials/scripts/gazebo.material</uri>
-            <name>Gazebo/Red</name>
-          </script>
-        </material>
-      </visual>
-    </gazebo>
-    <gazebo reference="uleg_1">
-      <visual>
-        <material>
-          <script>
-            <uri>file://media/materials/scripts/gazebo.material</uri>
-            <name>Gazebo/Red</name>
-          </script>
-        </material>
-      </visual>
-    </gazebo>
-    <gazebo reference="uleg_2">
-      <visual>
-        <material>
-          <script>
-            <uri>file://media/materials/scripts/gazebo.material</uri>
-            <name>Gazebo/Red</name>
-          </script>
-        </material>
-      </visual>
-    </gazebo>
-    <gazebo reference="uleg_3">
-      <visual>
-        <material>
-          <script>
-            <uri>file://media/materials/scripts/gazebo.material</uri>
-            <name>Gazebo/Red</name>
-          </script>
-        </material>
-      </visual>
-    </gazebo>
-    <gazebo reference="low_base">
-      <visual>
-        <material>
-          <script>
-            <uri>file://media/materials/scripts/gazebo.material</uri>
-            <name>Gazebo/Red</name>
-          </script>
-        </material>
-      </visual>
-    </gazebo>
-<!-- Patas unidas a los motors -->
-    <joint name="link_0_JOINT_1" type="revolute">
-      <origin xyz="0 -${1.717/6*length_base} 0" rpy="0 0 0"/>
-    	<parent link="link_0"/>
-    	<child link="uleg_1"/>
-      <limit effort="20" velocity="1.0" lower="-2.1" upper="2.1" />
-      <axis xyz="1 0 0"/>
-    </joint>
-    <joint name="link_0_JOINT_2" type="revolute">
-      <origin xyz="${-length_base/4} ${1.717/4*length_base-1.717/6*length_base+0.005} 0" rpy="0 0 ${4*PI/3}"/>
-    	<parent link="link_0"/>
-    	<child link="uleg_2"/>
-      <limit effort="20" velocity="1.0" lower="-2.1" upper="2.1" />
-      <axis xyz="1 0 0"/>
-    </joint>
-    <joint name="link_0_JOINT_3" type="revolute">
-      <origin xyz="${length_base/4} ${1.717/4*length_base-1.717/6*length_base} 0" rpy="0 0 ${2*PI/3}"/>
-    	<parent link="link_0"/>
-    	<child link="uleg_3"/>
-      <limit effort="20" velocity="1.0" lower="-2.1" upper="2.1" />
-      <axis xyz="1 0 0"/>
-    </joint>
-    <link name="uleg_1">
-      <inertial>
-        <origin xyz="0 ${-length_uleg/2+width_uleg/2+0.004}  0 " rpy="${PI/2} 0 0"/>
-        <mass value="${mass_uleg}"/>
-       	<xacro:default_inertial3 mass="${mass_uleg}" width="${length_uleg}" length="${width_uleg}" />
-      </inertial>
-      <visual>
-        <origin xyz="0 ${width_uleg/2+0.004} ${width_uleg/2+0.003} " rpy="${PI/2} ${PI} ${PI/2}"/>
-      	<geometry>
-          <mesh filename="package://delta_robot_support/urdf/meshes/upper_leg.STL" scale="0.001 0.001 0.001" />
-        </geometry>
-      </visual>
-      <collision>
-     	  <origin xyz="0 ${width_uleg/2+0.004} ${width_uleg/2} " rpy="${PI/2} ${PI} ${PI/2}"/>
-    	  <geometry>
-          <mesh filename="package://delta_robot_support/urdf/meshes/upper_leg.STL" scale="0.001 0.001 0.001" />
-        </geometry>
-      </collision>
-     </link>
-     <link name="uleg_2">
-      <inertial>
-           <origin xyz="0 ${-length_uleg/2+width_uleg/2+0.004}  0 " rpy="${PI/2} 0 0"/>
-           <mass value="${mass_uleg}"/>
-    	      <xacro:default_inertial3 mass="${mass_uleg}" width="${length_uleg}" length="${width_uleg}" />
-       </inertial>
-       <visual>
-         <origin xyz="0 ${width_uleg/2+0.004} ${width_uleg/2+0.003} " rpy="${PI/2} ${PI} ${PI/2}"/>
-    	   <geometry>
-           <mesh filename="package://delta_robot_support/urdf/meshes/upper_leg.STL" scale="0.001 0.001 0.001" />
-         </geometry>
-       </visual>
-       <collision>
-  	      <origin xyz="0 ${width_uleg/2+0.004} ${width_uleg/2} " rpy="${PI/2} ${PI} ${PI/2}"/>
-  	      <geometry>
-             <mesh filename="package://delta_robot_support/urdf/meshes/upper_leg.STL" scale="0.001 0.001 0.001" />
-         </geometry>
-       </collision>
-     </link>
-     <link name="uleg_3">
-       <inertial>
-           <origin xyz="0 ${-length_uleg/2+width_uleg/2+0.004}  0 " rpy="${PI/2} 0 0"/>
-           <mass value="${mass_uleg}"/>
-           <xacro:default_inertial3 mass="${mass_uleg}" width="${length_uleg}" length="${width_uleg}" />
-       </inertial>
-       <visual>
-         <origin xyz="0 ${width_uleg/2+0.004} ${width_uleg/2+0.003} " rpy="${PI/2} ${PI} ${PI/2}"/>
-       	 <geometry>
-           <mesh filename="package://delta_robot_support/urdf/meshes/upper_leg.STL" scale="0.001 0.001 0.001" />
-         </geometry>
-       </visual>
-        <collision>
-          <origin xyz="0 ${width_uleg/2+0.004} ${width_uleg/2} " rpy="${PI/2} ${PI} ${PI/2}"/>
-       	  <geometry>
-            <mesh filename="package://delta_robot_support/urdf/meshes/upper_leg.STL" scale="0.001 0.001 0.001" />
-          </geometry>
-        </collision>
-      </link>
-<!-- ****************************************************************** -->
-<!-- Brazo vertical de union con "upper_leg" 1 -->
-<!-- ****************************************************************** -->
-<!-- barilla horizontal de uninon entre "upper_leg" y la pata larga 1-->
+	<xacro:macro name="default_inertial2" params="mass length width">
+		<inertia ixx="${1/12*mass*(width*width+length*length)}" ixy="0.0" ixz="0.0"
+			iyy="${1/12*mass*(width*width+length*length)}" iyz="0.0"
+			izz="${1/12*mass*(width*width+width*width)}"/>
+	</xacro:macro>
+	<xacro:macro name="default_inertial3" params="mass length width">
+		<inertia ixx="${1/12*mass*(width*width+length*length)}" ixy="0.0" ixz="0.0"
+			 iyy="${1/12*mass*(width*width+length*length)}" iyz="0.0"
+			 izz="${1/12*mass*(length*length+length*length)}"/>
+	</xacro:macro>
+	<gazebo>
+		<plugin name="my_plugin" filename="libcontact.so"/>
+		<plugin filename="libgazebo_ros_control.so" name="gazebo_ros_control">
+			<robotNamespace>/${namespace}</robotNamespace>
+     		</plugin>
+		<self_collide>true</self_collide>
+		<enable_wind>false</enable_wind>
+  	</gazebo>
+	<link name="world"/>
+<!-- Visual Materials -->
+	<gazebo reference="link_0">
+		<visual><material><script>
+			<uri>file://media/materials/scripts/gazebo.material</uri>
+			<name>Gazebo/Red</name>
+		</script></material></visual>
+	</gazebo>
+	<gazebo reference="uleg_1">
+		<visual><material><script>
+			<uri>file://media/materials/scripts/gazebo.material</uri>
+			<name>Gazebo/Blue</name>
+		</script></material></visual>
+	</gazebo>
+	<gazebo reference="uleg_2">
+		<visual><material><script>
+			<uri>file://media/materials/scripts/gazebo.material</uri>
+			<name>Gazebo/Red</name>
+		</script></material></visual>
+	</gazebo>
+	<gazebo reference="uleg_3">
+		<visual><material><script>
+			<uri>file://media/materials/scripts/gazebo.material</uri>
+			<name>Gazebo/Red</name>
+		</script></material></visual>
+	</gazebo>
+	<gazebo reference="low_base">
+		<visual><material><script>
+			<uri>file://media/materials/scripts/gazebo.material</uri>
+			<name>Gazebo/Red</name>
+		</script></material></visual>
+	</gazebo>
+<!-- Fixed Base -->
+	<joint name="base" type="fixed">
+	  	<origin xyz="0 0 ${-distance_arm_uav+distance_ground}" rpy="0 0 0"/>
+	 	<parent link="world"/>
+	 	<child link="link_0"/>
+	</joint>
+	<gazebo reference="link_w_JOINT_w2">
+ 		<physics><ode>
+ 			<provide_feedback>true</provide_feedback>
+ 		</ode></physics>
+ 	</gazebo>
+	<link name="link_0">
+		<inertial>
+			<origin xyz="0 0 0" rpy="0 0 0"/>
+			<mass value="1"/>
+			<inertia ixx="1"  ixy="0"  ixz="0" iyy="1" iyz="0" izz="1" />
+		</inertial>
+		<visual>
+			<origin xyz="0 0 0" rpy="0 0 0"/>
+			<geometry>
+			<mesh filename="package://delta_robot_support/urdf/meshes/Base.stl" scale="0.001 0.001 0.001" />
+			</geometry>
+		</visual>
+		<collision>
+			<origin xyz="0 0 0" rpy="0 0 0"/>
+			<geometry>
+			<mesh filename="package://delta_robot_support/urdf/meshes/Base.stl" scale="0.001 0.001 0.001" />
+			</geometry>
+		</collision>
+	</link>
+<!-- Servo Joints -->
+	<joint name="link_0_JOINT_1" type="revolute">
+		<origin xyz="0 -${u} 0" rpy="0 0 0"/>
+		<parent link="link_0"/>
+		<child link="uleg_1"/>
+		<limit effort="20" velocity="1.0" lower="-2.1" upper="2.1" />
+		<axis xyz="1 0 0"/>
+	</joint>
+	<joint name="link_0_JOINT_2" type="revolute">
+		<origin xyz="${u*0.866} ${u*0.5} 0" rpy="0 0 ${2*PI/3}"/>
+		<parent link="link_0"/>
+		<child link="uleg_2"/>
+		<limit effort="20" velocity="1.0" lower="-2.1" upper="2.1" />
+		<axis xyz="1 0 0"/>
+	</joint>
+	<joint name="link_0_JOINT_3" type="revolute">
+		<origin xyz="${u*-0.866} ${u*0.5} 0" rpy="0 0 ${4*PI/3}"/>
+		<parent link="link_0"/>
+		<child link="uleg_3"/>
+		<limit effort="20" velocity="1.0" lower="-2.1" upper="2.1" />
+		<axis xyz="1 0 0"/>
+	</joint>
+<!-- Upper Legs -->
+	<link name="uleg_1">
+		<inertial>
+			<origin xyz="0 0 0 " rpy="${PI/2} 0 0"/>
+			<mass value="${mass_uleg}"/>
+			<xacro:default_inertial3 mass="${mass_uleg}" width="${length_uleg}" length="${width_uleg}" />
+		</inertial>
+		<visual>
+			<origin xyz="0 0 0 " rpy="${PI/2} ${PI} 0"/>
+			<geometry>
+			<mesh filename="package://delta_robot_support/urdf/meshes/Link1.stl" scale="0.001 0.001 0.001" />
+			</geometry>
+		</visual>
+		<collision>
+			<origin xyz="0 0 0 " rpy="${PI/2} ${PI} 0"/>
+			<geometry>
+			<mesh filename="package://delta_robot_support/urdf/meshes/Link1.stl" scale="0.001 0.001 0.001" />
+			</geometry>
+		</collision>
+	</link>
+	<link name="uleg_2">
+		<inertial>
+			<origin xyz="0 0 0 " rpy="${PI/2} 0 0"/>
+			<mass value="${mass_uleg}"/>
+			<xacro:default_inertial3 mass="${mass_uleg}" width="${length_uleg}" length="${width_uleg}" />
+		</inertial>
+		<visual>
+			<origin xyz="0 0 0" rpy="${PI/2} ${PI} 0"/>
+			<geometry>
+			<mesh filename="package://delta_robot_support/urdf/meshes/Link1.stl" scale="0.001 0.001 0.001" />
+			</geometry>
+		</visual>
+		<collision>
+			<origin xyz="0 0 0" rpy="${PI/2} ${PI} 0"/>
+			<geometry>
+			<mesh filename="package://delta_robot_support/urdf/meshes/Link1.stl" scale="0.001 0.001 0.001" />
+			</geometry>
+		</collision>
+	</link>
+	<link name="uleg_3">
+		<inertial>
+			<origin xyz="0 0 0 " rpy="${PI/2} 0 0"/>
+			<mass value="${mass_uleg}"/>
+			<xacro:default_inertial3 mass="${mass_uleg}" width="${length_uleg}" length="${width_uleg}" />
+		</inertial>
+		<visual>
+			<origin xyz="0 0 0" rpy="${PI/2} ${PI} 0"/>
+			<geometry>
+			<mesh filename="package://delta_robot_support/urdf/meshes/Link1.stl" scale="0.001 0.001 0.001" />
+			</geometry>
+		</visual>
+		<collision>
+			<origin xyz="0 0 0" rpy="${PI/2} ${PI} 0}"/>
+			<geometry>
+			<mesh filename="package://delta_robot_support/urdf/meshes/Link1.stl" scale="0.001 0.001 0.001" />
+			</geometry>
+		</collision>
+	</link>
+<!-- ****************************************************************** -->
+<!-- Vertical Connector with "upper_leg" 1 -->
+<!-- ****************************************************************** -->
+<!-- horizontal bar of connection between "upper_leg" and the long leg 1-->
       <joint name="uleg1_con" type="continuous">
     	   <origin xyz="0 -0.2 0" rpy="${PI/2-1.0358} 0 0"/>
@@ -234,5 +210,5 @@
         </collision>
        </link>
-<!-- barilla vertical larga 1 -->
+<!-- long vertical rod 1 -->
        <joint name="con_lleg_1" type="continuous">
          <origin xyz="-0.02 0 0" rpy="0 0 0"/>
@@ -260,5 +236,5 @@
            </collision>
        </link>
-<!-- barilla vertical 2 -->
+<!-- long vertical rod 2 -->
        <joint name="con2_lleg_1" type="continuous">
          <origin xyz="0.03 0 0" rpy="0 0 0"/>
@@ -549,5 +525,5 @@
             <origin xyz="-0.07 -0.015 -0.012" rpy="0 -0 0"/>
     	      <geometry>
-              <mesh filename="package://delta_robot_support/urdf/meshes/Platform.STL" scale="0.001 0.001 0.001" />
+              <mesh filename="package://delta_robot_support/urdf/meshes/EE.stl" scale="0.001 0.001 0.001" />
             </geometry>
           </visual>
