Commit message: Update delta_robot.urdf.xacro

File: delta_robot_support/urdf/delta_robot.urdf.xacro (robot description, xacro)
@@ -1,37 +1,46 @@
 <?xml version="1.0"?>
+<!--rostopic pub -1 /arms_joint_state_controller/command std_msgs/Float64MultiArray "{data:[0,1,-1],layout: {dim:[], data_offset: 1"}}-->
 <robot name="delta_robot" xmlns:xacro="http://www.ros.org/wiki/xacro">
-  	<xacro:property name="PI" value="3.1415926535897931"/>
-  	<xacro:property name="width" value="0.01" /> <!-- all links -->
-  	<xacro:property name="u" value="0.075" /> <!-- Radius of Base -->
-	<xacro:property name="ul" value="0.1" /> <!-- Length of Upper Leg -->
-	<xacro:property name="ll" value="0.15" /> <!-- Length of Lower Leg -->
-	<xacro:property name="e" value="0.05" /> <!-- Radius of EE -->
-	<xacro:property name="base_height" value="1" /> <!-- Length of Lower Leg -->
-	<xacro:property name="mass_uleg" value="0.0466" /> <!--upper leg mass-->
-  <xacro:property name="length_uleg" value="0.2" /> <!-- upper leg length -->
-  <xacro:property name="width_uleg" value="0.05" /> <!-- upper leg width -->
-  <xacro:property name="mass_lleg" value="0.04" /> <!-- low leg mass-->
-  <xacro:property name="length_lleg" value="0.2" /> <!-- low leg length-->
-  <xacro:property name="width_lleg" value="0.002" /> <!-- low leg width -->
-  <xacro:property name="mass_con" value="0.0173" /> <!-- connector mass-->
-	<xacro:property name="ULeg_mass" value="0.0483" /> <!-- EE mass-->
-	<xacro:property name="Base_mass" value="0.888"  /> <!-- EE mass-->
-	<xacro:property name="EE_mass"   value="0.0475" /> <!-- EE mass-->
-  <xacro:property name="namespace" value="delta_robot" />
-	<xacro:macro name="default_inertial2" params="mass length width">
-		<inertia ixx="${1/12*mass*(width*width+length*length)}" ixy="0.0" ixz="0.0"
-			iyy="${1/12*mass*(width*width+length*length)}" iyz="0.0"
-			izz="${1/12*mass*(width*width+width*width)}"/>
-	</xacro:macro>
-	<xacro:macro name="default_inertial3" params="mass length width">
-		<inertia ixx="${1/12*mass*(width*width+length*length)}" ixy="0.0" ixz="0.0"
-			 iyy="${1/12*mass*(width*width+length*length)}" iyz="0.0"
-			 izz="${1/12*mass*(length*length+length*length)}"/>
+  	<xacro:property name="namespace"    	value="delta_robot" />
+	<xacro:property name="PI"           	value="3.14159265358"/>
+	<xacro:property name="cosThirty"    	value="0.86602540378"/>
+	<xacro:property name="sinThirty"    	value="0.50000000000"/>
+	<xacro:property name="DegToRad"     	value="0.01745329251"/>
+	<xacro:property name="servo_max_force"  value="30"/>				<!-- Max force in N*ms of servos-->
+	<xacro:property name="servo_max_speed"  value="0.5"/>				<!-- Max angular velocity in rad/s of servos-->
+	<xacro:property name="servo_max_angle"  value="135"/>				<!-- Max angle from origin in degrees of servos-->
+	<xacro:property name="servo_min_angle"  value="-135"/>				<!-- Min angle from origin in degrees of servos-->
+	<xacro:property name="hip_angle"    	value="120.00000000000"/>	<!-- Starting angle of hip joints which becomes the origin during operation-->
+	<xacro:property name="knee_angle"   	value="109.23115703305"/>	<!-- Starting angle of knee joints-->
+	<xacro:property name="ankle_angle"  	value="130.76884296694"/>	<!-- Starting angle of ankle joints-->
+  	<xacro:property name="base_radius"  	value="0.075" /> 			<!-- Radius between center of base and hip joint in m-->
+	<xacro:property name="base_height"  	value="0.300" /> 			<!-- Z height of base with respect to ground in m-->
+	<xacro:property name="femur_x"      	value="0.040" /> 			<!-- Width in x direction of upper leg in m-->
+	<xacro:property name="femur_y"      	value="0.020" /> 			<!-- Width in y direction of upper leg in m-->
+	<xacro:property name="femur_z"      	value="0.100" /> 			<!-- Length of upper leg in m-->
+	<xacro:property name="femur_mass"   	value="0.049" /> 			<!-- Mass of upper leg in kg-->
+	<xacro:property name="tibia_x"      	value="0.009" /> 			<!-- Width in x direction of lower leg in m-->
+	<xacro:property name="tibia_y"      	value="0.009" /> 			<!-- Width in y direction of lower leg in m-->
+	<xacro:property name="tibia_z"      	value="0.150" /> 			<!-- Length of lower leg in m-->
+	<xacro:property name="tibia_mass"  		value="0.007" /> 			<!-- Mass of lower leg in kg-->
+	<xacro:property name="ee_radius"    	value="0.048" /> 			<!-- Radius between center of ee and ankle joint in m-->
+	<xacro:property name="ee_z"      		value="0.006" /> 			<!-- Height of ee in m-->
+	<xacro:property name="ee_mass"      	value="0.048" /> 			<!-- Mass of ee in kg-->
+	<xacro:property name="ankle_mass"   	value="0.005" /> 			<!-- Mass of each ball stud used in ankle joint in kg-->
+	<xacro:property name="ankle_radius" 	value="0.002" /> 			<!-- Radius of ankle joint in m-->
+	<xacro:property name="ankle_x"  		value="0.040" /> 			<!-- Width of ankle joint in m-->
+	<xacro:property name="knee_mass"    	value="0.005" /> 			<!-- Mass of each ball stud used in knee joint in kg-->
+	<xacro:property name="knee_radius"  	value="0.002" /> 			<!-- Radius of knee joint in m-->
+	<xacro:property name="knee_x"   		value="0.040" /> 			<!-- Width of knee joint in m-->
+	<xacro:macro name="inertia_rectangular" params="mass x y z">
+		<inertia ixx="${1/12*mass*(y*y+z*z)}" iyz="0.0"
+				 iyy="${1/12*mass*(x*x+z*z)}" ixz="0.0"
+		    	 izz="${1/12*mass*(x*x+y*y)}" ixy="0.0"/>
 	</xacro:macro>
 	<gazebo>
 		<plugin name="my_plugin" filename="libcontact.so"/>
 		<plugin filename="libgazebo_ros_control.so" name="gazebo_ros_control">
-			<robotNamespace>/${namespace}</robotNamespace>
-     		</plugin>
+		<robotNamespace>/${namespace}</robotNamespace>
+     	</plugin>
 		<self_collide>true</self_collide>
 		<enable_wind>false</enable_wind>
@@ -39,527 +48,582 @@
 	<link name="world"/>
 <!-- Visual Materials -->
-	<gazebo reference="link_0">
-		<visual><material><script>
-			<uri>file://media/materials/scripts/gazebo.material</uri>
-			<name>Gazebo/Red</name>
-		</script></material></visual>
-	</gazebo>
-	<gazebo reference="uleg_1">
-		<visual><material><script>
-			<uri>file://media/materials/scripts/gazebo.material</uri>
-			<name>Gazebo/Red</name>
-		</script></material></visual>
-	</gazebo>
-	<gazebo reference="uleg_2">
-		<visual><material><script>
-			<uri>file://media/materials/scripts/gazebo.material</uri>
-			<name>Gazebo/Red</name>
-		</script></material></visual>
-	</gazebo>
-	<gazebo reference="uleg_3">
-		<visual><material><script>
-			<uri>file://media/materials/scripts/gazebo.material</uri>
-			<name>Gazebo/Red</name>
-		</script></material></visual>
-	</gazebo>
-	<gazebo reference="low_base">
-		<visual><material><script>
-			<uri>file://media/materials/scripts/gazebo.material</uri>
-			<name>Gazebo/Red</name>
+	<gazebo reference="base">
+		<visual><material><script>
+			<uri>file://media/materials/scripts/gazebo.material</uri>
+			<name>Gazebo/DarkGrey</name>
+		</script></material></visual>
+	</gazebo>
+	<gazebo reference="femur_1">
+		<visual><material><script>
+			<uri>file://media/materials/scripts/gazebo.material</uri>
+			<name>Gazebo/DarkGrey</name>
+		</script></material></visual>
+	</gazebo>
+	<gazebo reference="femur_2">
+		<visual><material><script>
+			<uri>file://media/materials/scripts/gazebo.material</uri>
+			<name>Gazebo/DarkGrey</name>
+		</script></material></visual>
+	</gazebo>
+	<gazebo reference="femur_3">
+		<visual><material><script>
+			<uri>file://media/materials/scripts/gazebo.material</uri>
+			<name>Gazebo/DarkGrey</name>
+		</script></material></visual>
+	</gazebo>
+	<gazebo reference="tibia_1a">
+		<visual><material><script>
+			<uri>file://media/materials/scripts/gazebo.material</uri>
+			<name>Gazebo/DarkGrey</name>
+		</script></material></visual>
+	</gazebo>
+	<gazebo reference="tibia_1b">
+		<visual><material><script>
+			<uri>file://media/materials/scripts/gazebo.material</uri>
+			<name>Gazebo/DarkGrey</name>
+		</script></material></visual>
+	</gazebo>
+	<gazebo reference="tibia_2a">
+		<visual><material><script>
+			<uri>file://media/materials/scripts/gazebo.material</uri>
+			<name>Gazebo/DarkGrey</name>
+		</script></material></visual>
+	</gazebo>
+	<gazebo reference="tibia_2b">
+		<visual><material><script>
+			<uri>file://media/materials/scripts/gazebo.material</uri>
+			<name>Gazebo/DarkGrey</name>
+		</script></material></visual>
+	</gazebo>
+	<gazebo reference="tibia_3a">
+		<visual><material><script>
+			<uri>file://media/materials/scripts/gazebo.material</uri>
+			<name>Gazebo/DarkGrey</name>
+		</script></material></visual>
+	</gazebo>
+	<gazebo reference="tibia_3b">
+		<visual><material><script>
+			<uri>file://media/materials/scripts/gazebo.material</uri>
+			<name>Gazebo/DarkGrey</name>
+		</script></material></visual>
+	</gazebo>
+	<gazebo reference="ee">
+		<visual><material><script>
+			<uri>file://media/materials/scripts/gazebo.material</uri>
+			<name>Gazebo/DarkGrey</name>
 		</script></material></visual>
 	</gazebo>
 <!-- Fixed Base -->
-	<joint name="base" type="fixed">
+	<joint name="base_joint" type="fixed">
 	  	<origin xyz="0 0 ${base_height}" rpy="0 0 0"/>
 	 	<parent link="world"/>
-	 	<child link="link_0"/>
-	</joint>
-	<gazebo reference="link_w_JOINT_w2">
- 		<physics><ode>
- 			<provide_feedback>true</provide_feedback>
- 		</ode></physics>
- 	</gazebo>
-	<link name="link_0">
+	 	<child link="base"/>
+	</joint>
+	<link name="base">
 		<inertial>
 			<origin xyz="0 0 0" rpy="0 0 0"/>
 			<mass value="1"/>
-			<inertia ixx="1"  ixy="0"  ixz="0" iyy="1" iyz="0" izz="1" />
-		</inertial>
-		<visual>
-			<origin xyz="0 0 0" rpy="0 0 0"/>
-			<geometry>
-			<mesh filename="package://delta_robot_support/urdf/meshes/Base.stl" scale="0.001 0.001 0.001" />
-			</geometry>
-		</visual>
-		<collision>
-			<origin xyz="0 0 0" rpy="0 0 0"/>
-			<geometry>
-			<mesh filename="package://delta_robot_support/urdf/meshes/Base.stl" scale="0.001 0.001 0.001" />
-			</geometry>
-		</collision>
-	</link>
-<!-- Servo Joints -->
-	<joint name="link_0_JOINT_1" type="revolute">
-		<origin xyz="0 -${u} 0" rpy="0.522 0 0"/>
-		<parent link="link_0"/>
-		<child link="uleg_1"/>
-		<limit effort="20" velocity="1.0" lower="-2.1" upper="2.1" />
+			<inertia ixx="0" ixy="0" ixz="0" iyy="0" iyz="0" izz="0" />
+		</inertial>
+		<visual>
+			<origin xyz="0 0 0" rpy="0 0 0"/>
+			<geometry>
+			<mesh filename="package://delta_robot_support/urdf/meshes/Base_binary.stl" scale="0.001 0.001 0.001" />
+			</geometry>
+		</visual>
+		<collision>
+			<origin xyz="0 0 0" rpy="0 0 0"/>
+			<geometry>
+			<mesh filename="package://delta_robot_support/urdf/meshes/Base_binary.stl" scale="0.001 0.001 0.001" />
+			</geometry>
+		</collision>
+	</link>
+<!-- ********************************************************************** -->
+<!-- Hips							                                        -->
+<!-- ********************************************************************** -->
+	<joint name="hip_1" type="revolute">
+		<origin xyz="0 -${base_radius} 0" rpy="${hip_angle*DegToRad} 0 0"/>
+		<parent link="base"/>
+		<child link="femur_1"/>
+		<limit effort="${servo_max_force}" velocity="${servo_max_speed}" upper="${hip_angle+servo_max_angle}" lower="${hip_angle+servo_min_angle}"/>
 		<axis xyz="1 0 0"/>
-	</joint>
-	<joint name="link_0_JOINT_2" type="revolute">
-		<origin xyz="${u*0.866} ${u*0.5} 0" rpy="0.522 0 ${2*PI/3}"/>
-		<parent link="link_0"/>
-		<child link="uleg_2"/>
-		<limit effort="20" velocity="1.0" lower="-2.1" upper="2.1" />
+		<dynamics damping="0.1"/>
+	</joint>
+	<joint name="hip_2" type="revolute">
+		<origin xyz="${base_radius*cosThirty} ${base_radius*sinThirty} 0" rpy="${hip_angle*DegToRad} 0 ${120*DegToRad}"/>
+		<parent link="base"/>
+		<child link="femur_2"/>
+		<limit effort="${servo_max_force}" velocity="${servo_max_speed}" upper="${hip_angle+servo_max_angle}" lower="${hip_angle+servo_min_angle}"/>
 		<axis xyz="1 0 0"/>
-	</joint>
-	<joint name="link_0_JOINT_3" type="revolute">
-		<origin xyz="${u*-0.866} ${u*0.5} 0" rpy="0.522 0 ${4*PI/3}"/>
-		<parent link="link_0"/>
-		<child link="uleg_3"/>
-		<limit effort="20" velocity="1.0" lower="-2.1" upper="2.1" />
+		<dynamics damping="0.1"/>
+	</joint>
+	<joint name="hip_3" type="revolute">
+		<origin xyz="-${base_radius*cosThirty} ${base_radius*sinThirty} 0" rpy="${hip_angle*DegToRad} 0 ${240*DegToRad}"/>
+		<parent link="base"/>
+		<child link="femur_3"/>
+		<limit effort="${servo_max_force}" velocity="${servo_max_speed}" upper="${hip_angle+servo_max_angle}" lower="${hip_angle+servo_min_angle}"/>
 		<axis xyz="1 0 0"/>
-	</joint>
-<!-- Upper Legs -->
-	<link name="uleg_1">
-		<inertial>
-			<origin xyz="0 0 0 " rpy="${PI/2} 0 0"/>
-			<mass value="${mass_uleg}"/>
-			<xacro:default_inertial3 mass="${mass_uleg}" width="${length_uleg}" length="${width_uleg}" />
-		</inertial>
-		<visual>
-			<origin xyz="0 0 0 " rpy="${PI/2} ${PI} 0"/>
-			<geometry>
-			<mesh filename="package://delta_robot_support/urdf/meshes/Link1.stl" scale="0.001 0.001 0.001" />
-			</geometry>
-		</visual>
-		<collision>
-			<origin xyz="0 0 0 " rpy="${PI/2} ${PI} 0"/>
-			<geometry>
-			<mesh filename="package://delta_robot_support/urdf/meshes/Link1.stl" scale="0.001 0.001 0.001" />
-			</geometry>
-		</collision>
-	</link>
-	<link name="uleg_2">
-		<inertial>
-			<origin xyz="0 0 0" rpy="${PI/2} 0 0"/>
-			<mass value="${mass_uleg}"/>
-			<xacro:default_inertial3 mass="${mass_uleg}" width="${length_uleg}" length="${width_uleg}" />
-		</inertial>
-		<visual>
-			<origin xyz="0 0 0" rpy="${PI/2} ${PI} 0"/>
-			<geometry>
-			<mesh filename="package://delta_robot_support/urdf/meshes/Link1.stl" scale="0.001 0.001 0.001" />
-			</geometry>
-		</visual>
-		<collision>
-			<origin xyz="0 0 0" rpy="${PI/2} ${PI} 0"/>
-			<geometry>
-			<mesh filename="package://delta_robot_support/urdf/meshes/Link1.stl" scale="0.001 0.001 0.001" />
-			</geometry>
-		</collision>
-	</link>
-	<link name="uleg_3">
-		<inertial>
-			<origin xyz="0 0 0" rpy="${PI/2} 0 0"/>
-			<mass value="${mass_uleg}"/>
-			<xacro:default_inertial3 mass="${mass_uleg}" width="${length_uleg}" length="${width_uleg}" />
-		</inertial>
-		<visual>
-			<origin xyz="0 0 0" rpy="${PI/2} ${PI} 0"/>
-			<geometry>
-			<mesh filename="package://delta_robot_support/urdf/meshes/Link1.stl" scale="0.001 0.001 0.001" />
-			</geometry>
-		</visual>
-		<collision>
-			<origin xyz="0 0 0" rpy="${PI/2} ${PI} 0"/>s
-			<geometry>
-			<mesh filename="package://delta_robot_support/urdf/meshes/Link1.stl" scale="0.001 0.001 0.001" />
-			</geometry>
-		</collision>
-	</link>
+		<dynamics damping="0.1"/>
+	</joint>
 <!-- ********************************************************************** -->
-<!-- Vertical Connector with "upper_leg" 1                                  -->
+<!-- Femurs							                                        -->
 <!-- ********************************************************************** -->
-<!-- horizontal bar of connection between "upper_leg1" and "lower_leg1ab"   -->
-	<joint name="uleg_1_to_elbow" type="continuous">
-		<origin xyz="0 -${ul} 0" rpy="0.3178 0 0"/>
-		<parent link="uleg_1"/>
-		<child link="leg1_elbow"/>
+	<link name="femur_1">
+		<inertial>
+			<origin xyz="0 0 ${femur_z/2}" rpy="0 0 0"/>
+			<mass value="${femur_mass}"/>
+			<xacro:inertia_rectangular mass="${femur_mass}" x="${femur_x}" y="${femur_y}" z="${femur_z}" />
+		</inertial>
+		<visual>
+			<origin xyz="0 0 0" rpy="0 0 0"/>
+			<geometry>
+			<mesh filename="package://delta_robot_support/urdf/meshes/Femur_binary.stl" scale="0.001 0.001 0.001" />
+			</geometry>
+		</visual>
+		<collision>
+			<origin xyz="0 0 0" rpy="0 0 0"/>
+			<geometry>
+			<mesh filename="package://delta_robot_support/urdf/meshes/Femur_binary.stl" scale="0.001 0.001 0.001" />
+			</geometry>
+		</collision>
+	</link>
+	<link name="femur_2">
+		<inertial>
+			<origin xyz="0 0 ${femur_z/2}" rpy="0 0 0"/>
+			<mass value="${femur_mass}"/>
+			<xacro:inertia_rectangular mass="${femur_mass}" x="${femur_x}" y="${femur_y}" z="${femur_z}" />
+		</inertial>
+		<visual>
+			<origin xyz="0 0 0" rpy="0 0 0"/>
+			<geometry>
+			<mesh filename="package://delta_robot_support/urdf/meshes/Femur_binary.stl" scale="0.001 0.001 0.001" />
+			</geometry>
+		</visual>
+		<collision>
+			<origin xyz="0 0 0" rpy="0 0 0"/>
+			<geometry>
+			<mesh filename="package://delta_robot_support/urdf/meshes/Femur_binary.stl" scale="0.001 0.001 0.001" />
+			</geometry>
+		</collision>
+	</link>
+	<link name="femur_3">
+		<inertial>
+			<origin xyz="0 0 ${femur_z/2}" rpy="0 0 0"/>
+			<mass value="${femur_mass}"/>
+			<xacro:inertia_rectangular mass="${femur_mass}" x="${femur_x}" y="${femur_y}" z="${femur_z}" />
+		</inertial>
+		<visual>
+			<origin xyz="0 0 0" rpy="0 0 0"/>
+			<geometry>
+			<mesh filename="package://delta_robot_support/urdf/meshes/Femur_binary.stl" scale="0.001 0.001 0.001" />
+			</geometry>
+		</visual>
+		<collision>
+			<origin xyz="0 0 0" rpy="0 0 0"/>
+			<geometry>
+			<mesh filename="package://delta_robot_support/urdf/meshes/Femur_binary.stl" scale="0.001 0.001 0.001" />
+			</geometry>
+		</collision>
+	</link>
+<!-- ********************************************************************** -->
+<!-- Knees							                                        -->
+<!-- ********************************************************************** -->
+	<joint name="femur_1_to_knee_1" type="continuous">
+		<origin xyz="0 0 ${femur_z}" rpy="${knee_angle*DegToRad} 0 0"/>
+		<parent link="femur_1"/>
+		<child link="knee_1"/>
 		<axis xyz="1 0 0"/>
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